File: kicad/Evaluation_Board_v1/EVAL-SCS001V1_Official.kicad_sch (KiCad schematic)
At the start: 17 parts, among them J1 Screw_Terminal_01x02, J2 GSB1C211110DS1HR, U1 STL6P3LLH6, U2 STUSB4500QTR

Commit message: Update KiCad schematic
Added component names and values corresponding to the datasheet.
Parts:
- C1, C2: value C -> 1uF
- C12: renamed from C3; value C -> 100nF
- R1: renamed from R6; value R -> 1k
- R10: renamed from R7; value R -> 100k
- R11: renamed from R3; value R -> 22k
- R12: renamed from R5; value R -> 100R
- R2: renamed from R4; value R -> 1k
- R20: renamed from R1; value R -> 22k
- R21: renamed from R2; value R -> 22k
Changed lines of the file:
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@@
 		(dnp no)
 		(fields_autoplaced yes)
-		(property "Reference" "R1"
+		(property "Reference" "R20"
 			(at 227.33 116.8399 0)
 			(effects
@@
 			)
 		)
-		(property "Value" "R"
+		(property "Value" "22k"
 			(at 227.33 119.3799 0)
 			(effects
@@
 			(project ""
 				(path "/cc1f831b-8f89-4c01-ad4b-13a86b2cf79d"
-					(reference "R1")
+					(reference "R20")
 					(unit 1)
 				)
@@
 		(dnp no)
 		(fields_autoplaced yes)
-		(property "Reference" "R3"
+		(property "Reference" "R11"
 			(at 190.5 64.7699 0)
 			(effects
@@
 			)
 		)
-		(property "Value" "R"
+		(property "Value" "22k"
 			(at 190.5 67.3099 0)
 			(effects
@@
 			(project ""
 				(path "/cc1f831b-8f89-4c01-ad4b-13a86b2cf79d"
-					(reference "R3")
+					(reference "R11")
 					(unit 1)
 				)
@@
 		(dnp no)
 		(fields_autoplaced yes)
-		(property "Reference" "R6"
+		(property "Reference" "R1"
 			(at 147.32 62.2299 0)
 			(effects
@@
 			)
 		)
-		(property "Value" "R"
+		(property "Value" "1k"
 			(at 147.32 64.7699 0)
 			(effects
@@
 			(project ""
 				(path "/cc1f831b-8f89-4c01-ad4b-13a86b2cf79d"
-					(reference "R6")
+					(reference "R1")
 					(unit 1)
 				)
@@
 		(dnp no)
 		(fields_autoplaced yes)
-		(property "Reference" "C3"
+		(property "Reference" "C12"
 			(at 210.82 52.07 90)
 			(effects
@@
 			)
 		)
-		(property "Value" "C"
+		(property "Value" "100nF"
 			(at 210.82 54.61 90)
 			(effects
@@
 			(project ""
 				(path "/cc1f831b-8f89-4c01-ad4b-13a86b2cf79d"
-					(reference "C3")
+					(reference "C12")
 					(unit 1)
 				)
@@
 		(dnp no)
 		(fields_autoplaced yes)
-		(property "Reference" "R5"
+		(property "Reference" "R12"
 			(at 200.66 53.34 90)
 			(effects
@@
 			)
 		)
-		(property "Value" "R"
+		(property "Value" "100R"
 			(at 200.66 55.88 90)
 			(effects
@@
 			(project ""
 				(path "/cc1f831b-8f89-4c01-ad4b-13a86b2cf79d"
-					(reference "R5")
+					(reference "R12")
 					(unit 1)
 				)
@@
 		(on_board yes)
 		(dnp no)
-		(fields_autoplaced yes)
-		(property "Reference" "R7"
-			(at 190.5 52.0699 0)
-			(effects
-				(font
-					(size 1.27 1.27)
-				)
-				(justify left)
-			)
-		)
-		(property "Value" "R"
-			(at 190.5 54.6099 0)
+		(property "Reference" "R10"
+			(at 189.23 52.07 0)
+			(effects
+				(font
+					(size 1.27 1.27)
+				)
+				(justify left)
+			)
+		)
+		(property "Value" "100k"
+			(at 189.23 54.102 0)
 			(effects
 				(font
@@
 			(project ""
 				(path "/cc1f831b-8f89-4c01-ad4b-13a86b2cf79d"
-					(reference "R7")
+					(reference "R10")
 					(unit 1)
 				)
@@
 		(dnp no)
 		(fields_autoplaced yes)
-		(property "Reference" "R2"
+		(property "Reference" "R21"
 			(at 237.49 116.8399 0)
 			(effects
@@
 			)
 		)
-		(property "Value" "R"
+		(property "Value" "22k"
 			(at 237.49 119.3799 0)
 			(effects
@@
 			(project ""
 				(path "/cc1f831b-8f89-4c01-ad4b-13a86b2cf79d"
-					(reference "R2")
+					(reference "R21")
 					(unit 1)
 				)
@@
 		(on_board yes)
 		(dnp no)
-		(fields_autoplaced yes)
 		(property "Reference" "C2"
-			(at 171.45 86.36 90)
-			(effects
-				(font
-					(size 1.27 1.27)
-				)
-			)
-		)
-		(property "Value" "C"
-			(at 171.45 88.9 90)
+			(at 174.498 90.932 90)
+			(effects
+				(font
+					(size 1.27 1.27)
+				)
+			)
+		)
+		(property "Value" "1uF"
+			(at 174.752 92.964 90)
 			(effects
 				(font
@@
 			)
 		)
-		(property "Value" "C"
+		(property "Value" "1uF"
 			(at 171.45 82.55 90)
 			(effects
@@
 		(dnp no)
 		(fields_autoplaced yes)
-		(property "Reference" "R4"
+		(property "Reference" "R2"
 			(at 220.98 64.7699 0)
 			(effects
@@
 			)
 		)
-		(property "Value" "R"
+		(property "Value" "1k"
 			(at 220.98 67.3099 0)
 			(effects
@@
 			(project ""
 				(path "/cc1f831b-8f89-4c01-ad4b-13a86b2cf79d"
-					(reference "R4")
-					(unit 1)
-				)
+					(reference "R2")
+					(unit 1)
+				)

Commit message: Reuploaded revised schematic
Added test points and connections to USB-C connector symbol.
Parts:
- added C50: 4.7uF, symbol Device:C
- added CR3: ESDA25P35-1U1M, QFN1610_STM, symbol ESDA25P35:ESDA25P35-1U1M
- added TP1, TP2, TP3, TP4, TP5, TP6, TP7, TP8: TestPoint_Small, symbol Connector:TestPoint_Small
Connections:
- net VBUS_B is gone; now on net VBUS_A: J2.B4 (VBUS_B), J2.B9 (VBUS_B)
- net GND: now also J2.SH1 (SHIELD), J2.SH2 (SHIELD), J2.SH3 (SHIELD), J2.SH4 (SHIELD), C50.2, CR3.2, TP7.1
- net VBUS_A: now also R1.1, R10.1, U1.1 (S), U1.2 (S), U1.3 (S), U2.24 (VDD), C50.1, CR3.1, TP1.1
- net at C12.1, CR2.1, D1.4 (A)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: now also TP8.1
- net at CR1.1, J2.B5 (CC2), U2.4 (CC2)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: now also TP5.1
- net at CR1.2, J2.A5 (CC1), U2.1 (CC1DB)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: now also TP6.1
- net at C2.2, U2.23 (VREG_2V7): now also TP2.1
- net at U2.7 (SCL): now also TP3.1
- net at U2.8 (SDA): now also TP4.1
Other:
- moved on the sheet: J2
